Commit message: updating the env for fer

File: hpp_control/robots/fer.urdf (robot description, URDF)
Before this commit: robot fer, 14 links, 13 joints
Links:
- added link panda1_box, mass 100; collision box size=0.803 0.44 0.80; visual box size=0.803 0.44 0.80
- added link support_link, mass 200; collision box size=0.3 0.3 0.02; collision box size=1.703 0.803 0.76
- added link wall_link_1, mass 200; collision box size=3.0 0.1 2.0; visual box size=3.0 0.1 2.0
- added link wall_link_2, mass 200; collision box size=0.1 2.0 2.0; visual box size=0.1 2.0 2.0
- added link wall_link_3, mass 200; collision box size=0.7 0.12 2.0; visual box size=0.7 0.12 2.0
Joints:
- added joint panda1_box_joint: type fixed, parent world, child panda1_box, origin xyz=0.45 -0.18 1.17
- added joint support_joint: type fixed, parent support_link, child fer_link0, origin xyz=0.718 -0.1655 .78 rpy=0 0 0
- added joint wall_joint_1: type fixed, parent world, child wall_link_1, origin xyz=0 1.07 0
- added joint wall_joint_2: type fixed, parent world, child wall_link_2, origin xyz=1.78 0 0
- added joint wall_joint_3: type fixed, parent world, child wall_link_3, origin xyz=1.40 0.96 0
- joint world_joint: child fer_link0 -> support_link; origin xyz=0 0 0 rpy=0 0 0 -> xyz=0 0 0 rpy=0 0 3.141592653589793
