Commit message: add fr3 env + cleaning

File: hpp_control/urdf/fr3.urdf (robot description, URDF)
Before this commit: robot fr3, 14 links, 13 joints
Links:
- added link panda1_box, mass 100; collision box size=0.803 0.44 0.80; visual box size=0.803 0.44 0.80
- added link support_link, mass 200; collision box size=0.3 0.3 0.02; collision box size=1.703 0.803 0.76
- added link wall_link_1, mass 200; collision box size=3.0 0.1 2.0; visual box size=3.0 0.1 2.0
- added link wall_link_2, mass 200; collision box size=0.1 2.0 2.0; visual box size=0.1 2.0 2.0
- added link wall_link_3, mass 200; collision box size=0.7 0.12 2.0; visual box size=0.7 0.12 2.0
Joints:
- added joint panda1_box_joint: type fixed, parent world, child panda1_box, origin xyz=-0.7 0.18 1.17
- added joint support_joint: type fixed, parent support_link, child fr3_link0, origin xyz=0.563 -0.1655 .78 rpy=0 0 3.141592653589793
- added joint wall_joint_1: type fixed, parent world, child wall_link_1, origin xyz=0 1.07 0
- added joint wall_joint_2: type fixed, parent world, child wall_link_2, origin xyz=1.78 0 0
- added joint wall_joint_3: type fixed, parent world, child wall_link_3, origin xyz=1.40 0.96 0
- joint world_joint: child fr3_link0 -> support_link

Commit message: fix bugs without docker

File: hpp_control/urdf/fr3.urdf (robot description, URDF)
Before this commit: robot fr3, 19 links, 18 joints
Joints:
- joint fr3_joint1: limit lower=-2.7437 upper=2.7437 effort=87.0 velocity=0.9 -> lower=-2.7437 upper=2.7437 effort=87.0 velocity=2.62
- joint fr3_joint2: limit lower=-1.7837 upper=1.7837 effort=87.0 velocity=0.9 -> lower=-1.7837 upper=1.7837 effort=87.0 velocity=2.62
- joint fr3_joint3: limit lower=-2.9007 upper=2.9007 effort=87.0 velocity=0.9 -> lower=-2.9007 upper=2.9007 effort=87.0 velocity=2.62
- joint fr3_joint4: limit lower=-3.0421 upper=-0.1518 effort=87.0 velocity=0.9 -> lower=-3.0421 upper=-0.1518 effort=87.0 velocity=2.62
- joint fr3_joint5: limit lower=-2.8065 upper=2.8065 effort=12.0 velocity=0.9 -> lower=-2.8065 upper=2.8065 effort=12.0 velocity=2.62
- joint fr3_joint6: limit lower=0.5445 upper=4.5169 effort=12.0 velocity=0.9 -> lower=0.5445 upper=4.5169 effort=12.0 velocity=2.62
- joint fr3_joint7: limit lower=-3.0159 upper=3.0159 effort=12.0 velocity=0.9 -> lower=-3.0159 upper=3.0159 effort=12.0 velocity=2.62

Commit message: work on bigg

File: hpp_control/urdf/fr3.urdf (robot description, URDF)
Before this commit: robot fr3, 19 links, 18 joints
Links:
- removed link wall_link_2
- removed link wall_link_3
Joints:
- removed joint wall_joint_2
- removed joint wall_joint_3
- joint panda1_box_joint: origin xyz=-0.7 0.18 1.17 -> xyz=-0.7 0.18 0.4
- joint support_joint: origin xyz=0.563 -0.1655 .78 rpy=0 0 3.141592653589793 -> xyz=0.563 -0.1655 0 rpy=0 0 3.141592653589793

Commit message: adding box in urdf

File: hpp_control/urdf/fr3.urdf (robot description, URDF)
Before this commit: robot fr3, 17 links, 16 joints
Links:
- added link box_link_1, mass 200; collision box size=0.02 0.35 0.2; collision box size=0.02 0.35 0.2
Joints:
- added joint box_joint_1: type fixed, parent world, child box_link_1, origin xyz=0.85 0.26 0.1

Commit message: working on demos

File: hpp_control/urdf/fr3.urdf (robot description, URDF)
Before this commit: robot fr3, 18 links, 17 joints
Links:
- removed link box_link_1
Joints:
- removed joint box_joint_1
