Commit message: Fix script move_one_box

File: hpp_control/urdf/fer.urdf (robot description, URDF)
Before this commit: robot fer, 19 links, 18 joints
Joints:
- joint support_joint: origin xyz=0.718 -0.1655 .78 rpy=0 0 0 -> xyz=0.568 -0.1655 .78 rpy=0 0 3.14156

Commit message: code version for rss2026

File: hpp_control/urdf/fer.urdf (robot description, URDF)
Before this commit: robot fer, 19 links, 18 joints
Links:
- removed link panda1_box
Joints:
- removed joint panda1_box_joint
